File: RCCM_ESP32mini/RCCM_ESP32mini.sch (KiCad schematic (older format))
At the start: 14 parts, among them CN1 Conn_02x04_Odd_Even, CN2 Conn_01x08, CN3 Conn_01x07, CN4 Conn_01x06, CN5 Conn_01x06, CN6 Conn_02x10_Odd_Even, CN7 Conn_02x10_Odd_Even, CN8 Conn_01x06, J1 Conn_01x02, U1 LT1129-3.3_SOT223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

Commit message: Gerber change
Parts:
- added J2: Conn_01x02, Pin_Headers:Pin_Header_Straight_2x01_Pitch2.54mm, symbol Conn_01x02
Connections:
- net GND: now also J2.2 (Pin_2)
- net MODEd: now also J2.1 (Pin_1)
Changed lines of the file:
@@
 	5650 4450 5650 4350
 Connection ~ 5650 4350
+Text GLabel 3300 3250 0    60   Input ~ 0
+MODEd
+Wire Wire Line
+	3300 3250 3400 3250
+$Comp
+L Conn_01x02 J2
+U 1 1 5EC22177
+P 3600 3250
+F 0 "J2" H 3600 3350 50  0000 C CNN
+F 1 "Conn_01x02" H 3600 3050 50  0000 C CNN
+F 2 "Pin_Headers:Pin_Header_Straight_2x01_Pitch2.54mm" H 3600 3250 50  0001 C CNN
+F 3 "" H 3600 3250 50  0001 C CNN
+	1    3600 3250
+	1    0    0    -1
+$EndComp
+Text GLabel 3300 3350 0    60   Input ~ 0
+GND
+Wire Wire Line
+	3300 3350 3400 3350
 $EndSCHEMATC

Commit message: SDx Update
(No:Pos:SDx:CNx:Nano:ESP32:M5S),
(S1:LEFT:SD0:CN1-5:No14:IO19:NC),
(S2:CEN:SD1:CN1-3:No15:IO18:G32),
(S3:RIGHT:SD2:CN1-1:No16:IO5:G33)
Connections:
- net IO05: now also CN1.1 (Pin_1), CN6.14 (Pin_14); no longer CN1.5 (Pin_5)
- net IO19: now also CN1.5 (Pin_5); no longer CN1.1 (Pin_1)
- no-connect marks 4 -> 3
Changed lines of the file:
@@
 Text GLabel 5400 2700 2    60   Input ~ 0
 SCL
-Text GLabel 4500 2900 0    60   Input ~ 0
+Text GLabel 4500 2700 0    60   Input ~ 0
 SD0
 Text GLabel 4500 2800 0    60   Input ~ 0
 SD1
-Text GLabel 4500 2700 0    60   Input ~ 0
+Text GLabel 4500 2900 0    60   Input ~ 0
 SD2
 Wire Wire Line
@@
 Text Notes 4400 3150 0    60   ~ 0
 to RC Car
-NoConn ~ 5400 1700
 $Comp
 L KA378R33 U2
@@
 Wire Wire Line
 	3300 3350 3400 3350
+Text GLabel 5400 1700 2    60   Input ~ 0
+IO05
 $EndSCHEMATC
