File: RCCM_RPiZW/RCCM_RPiZW.kicad_pcb (KiCad board)
At the start: 2 copper layers, 45.7 x 92.7 mm, 31 parts, among them CN1 Conn_02x20_Odd_Even, CN2 Conn_02x04_Odd_Even, CN3 Conn_01x08, CN4 Conn_01x06, CN5 Conn_01x07, CN6 Conn_01x06, IC1 LP2950-3.0_TO92, J1 Conn_01x02, J2 Conn_01x02

Commit message: Update RPiZW Gerber
Parts:
- added DC1-5: Conn_01x01, Pin_Headers:Pin_Header_Straight_1x01_Pitch2.54mm, F.Cu at (95.2, 73.0)
- added DC1-6: Conn_01x01, Pin_Headers:Pin_Header_Straight_1x01_Pitch2.54mm, F.Cu at (99.1, 71.1)
- added DC1-7: Conn_01x01, Pin_Headers:Pin_Header_Straight_1x01_Pitch2.54mm, F.Cu at (109.9, 73.0)
- added DC1-8: Conn_01x01, Pin_Headers:Pin_Header_Straight_1x01_Pitch2.54mm, F.Cu at (106.0, 71.1)
- moved DC1-3 30.4 mm to (109.9, 99.7)
- moved DC1-4 29.2 mm to (106.0, 101.6)
- moved J1 21.9 mm to (95.2, 87.6), turned to 90 degrees
- moved DC1-2 7.73 mm to (99.1, 101.6)
- moved DC1-1 1.42 mm to (95.2, 99.7)
- moved H5 1.27 mm to (137.2, 40.6)
- moved H6 1.27 mm to (96.5, 40.6)
- moved C1 0.64 mm to (102.2, 117.5)
Connections:
- DC1-2 pad 1: GND -> VBat
- DC1-3 pad 1: +5V -> GND
Routing:
- net GND: track 0.00 -> 327.2 mm
- net 3V3: track 0.00 -> 207.7 mm
- net VBat: track 0.00 -> 117.0 mm
- net GP03: track 0.00 -> 103.3 mm
- net BIN2: track 0.00 -> 98.0 mm
- net GP02: track 0.00 -> 91.2 mm
- net +5V: track 0.00 -> 75.9 mm
- net AIN2: track 0.00 -> 72.5 mm
- net AIN1: track 0.00 -> 70.5 mm
- net BIN1: track 0.00 -> 67.0 mm
- net GP22: track 0.00 -> 61.4 mm
- net GP25: track 0.00 -> 59.2 mm
- net GP23: track 0.00 -> 58.3 mm
- net GP26: track 0.00 -> 58.1 mm, vias 0 -> 1
- net GP24: track 0.00 -> 55.6 mm
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- added copper zone on B.Cu, net GND
- added copper zone on F.Cu, net GND
Other:
- board size 45.7 x 92.7 mm -> 45.7 x 94 mm
- net class MTR added: clearance 0.3, trace_width 1.7, via_dia 0.6, via_drill 0.4
- net class POW added: clearance 0.2, trace_width 0.4, via_dia 0.6, via_drill 0.4
