File: RCCM_M5StickC_a/RCCM_M5StickC.kicad_pcb (KiCad board)
At the start: 2 copper layers, 24.1 x 44.5 mm, 16 parts, among them CN1 Conn_02x04_Odd_Even, CN2 Conn_01x04, CN3 Conn_01x04, CN4 Conn_01x08

Commit message: Small changes
M5Stick-C Rev.a
ESP32 None
RasPi ZW  Change gerber
Parts:
- removed H2, H4: MountingHole_3.5mm, Mounting_Holes:MountingHole_3.5mm
- moved CN3 3.81 mm to (81.3, 81.9), turned to 155 degrees
- moved CN2 3.17 mm to (81.3, 47.6), turned to 205 degrees
Routing:
- net GND: track 80.8 -> 139.1 mm
- net G00: track 56.3 -> 81.0 mm
- net G33: track 28.9 -> 43.1 mm
- net G32: track 42.3 -> 43.7 mm
- net G26: track 64.6 -> 64.0 mm
