File: RCCM_ESP32mini_a/RCCM_ESP32mini.kicad_pcb (KiCad board)
At the start: 2 copper layers, 38.1 x 49.5 mm, 20 parts, among them CN1 Conn_02x04_Odd_Even, CN2 Conn_01x08, CN3 Conn_01x07, CN4 Conn_01x06, CN5 Conn_01x06, CN6 Conn_02x10_Odd_Even, CN7 Conn_02x10_Odd_Even, CN8 Conn_01x06, J1 Conn_01x02, J2 Conn_01x02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

Commit message: Rev.A
Parts:
- moved CN2 2.54 mm to (81.3, 53.3)
Routing:
- net Vin: track 95.1 -> 70.0 mm
- net GND: track 156.3 -> 134.0 mm, vias 7 -> 5
- net AIN2: track 44.2 -> 38.8 mm
- net BIN2: track 56.9 -> 54.4 mm
- net BIN1: track 63.7 -> 61.1 mm
- net AIN1: track 52.1 -> 49.5 mm
- net VCCe: track 48.6 -> 47.9 mm
